File: io_board.kicad_sch (KiCad schematic)
At the start: 133 parts, among them J1 Conn_02x04_Top_Bottom, J10 JST-GH 4Pin, J13 Conn_02x03_Odd_Even, J15 USB_C_Receptacle_USB2.0, J16 TC2050, J2 Conn_02x04_Top_Bottom, J3 Conn_02x03_Odd_Even, J4 SWD, J5 JST-GH 4Pin, J6 JST-GH 4Pin, J7 JST-GH 4Pin, J8 JST-GH 4Pin, J9 JST-GH 4Pin, SW1 KMR721NGLFS, SW2 KMR721NGLFS, SW3 KMR721NGLFS, U1 171050601, U2 STM32F105RCTx, U3 AZ1117-3.3, U4 W25Q128JVP, U5 MCP2562-E-SN, U6 MCP2562-E-SN, Y1 8MHz 12pF

Commit message: add comment for i_sense 1 and 2
Other:
- note added: "HCO12"
- note added: "HCO34"
Changed lines of the file:
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@@
+		)
+	)
+	(text "HCO34"
+		(exclude_from_sim no)
+		(at 370.84 45.72 0)
+		(effects
+			(font
+				(size 1.27 1.27)
+			)
 		)
 	)
@@
 		)
 	)
+	(text "HCO12"
+		(exclude_from_sim no)
+		(at 371.094 48.26 0)
+		(effects
+			(font
+				(size 1.27 1.27)
+			)
+		)
+	)
